File: PCB/MCU-STM32F446RET6.sch (KiCad schematic (older format))
At the start: 41 parts, among them J3 20021121-00010C4LF, J4 0475890001-MicroUSBPort, P1 CONN_01X20, P2 CONN_01X20, SW1 B3U-1000P, U3 STM32F446RET6_-_TQFP64, X1 ABM3B8.000MHZB2T, X2 ABS07-32.768KHZ-9-T

Commit message: Schematic Done, Board Underway
Schematic completed. STM32 section upated from Aria project schematic,
ESP32 schematic completed with the help of reference schematic.
Datasheets for componens used also added. The PCB is near complete, Aria
was improted and modifed to speed up the process. More to come!
Parts:
- removed P1, P2: CONN_01X20, Pin_Headers:Pin_Header_Straight_1x20, symbol CONN_01X20
- added FD1, FD2, FD3: FIDUCIAL, PCB_Footprints:FIDUCIAL, symbol FIDUCIAL
- added H1, H2, H3, H4: M2.5_Hole, PCB_Footprints:M2.5_HOLE, symbol M2.5_Hole
- added P1, P2: CONN_01X18, symbol CONN_01X18
Connections:
- net labels added: PA10, PA11, PA12, PA3, PA4, PA5, PA6, PA7, PA8, PA9, PB0, PB1, PB10, PB5, PB6, PB7, PB8, PB9, PC0, PC1, PC10, PC11, PC12, PC13, PC4, PC5, PC6, PC7, PC8, PC9
- wire segments 103 -> 172
- no-connect marks 0 -> 7
Other:
- moved on the sheet: C10, C11, C12, C13, C4, C5, C6, C7, C8, C9, FB1, J3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
