File: PCB/_saved_WiFi-BLE-ESP32.sch (KiCad schematic (older format))
At the start: 27 parts, among them T1 1909763-1, U4 ESP32, U5 W25Q64FWSSIG, X3 FA-128_26.0000MF10Z-AC3

Commit message: PCB
PCB done
Parts:
- removed C23, C25, C26: CL05B104JP5NNNC, PCB_Footprints:C0402, symbol CL05B104JP5NNNC
- added C23, C25: CL10A106KQ8NNNC, PCB_Footprints:C0603, symbol CL10A106KQ8NNNC
Connections:
- net +3V3: now also C23.1, C25.1
- net GND: now also C23.2, C25.2
Other:
- moved on the sheet: C21, C22, C28
