File: PCB - ESP3212/WiFi-BLE-ESP32.sch (KiCad schematic (older format))
At the start: 2 parts, among them U4 ESP3212

Commit message: Tweaks, DRC cleared, images, readme
Tweaked both designs according to the dev board scheamtics provided by
Espressif in the datasheets folder. Cleared both boards of DRC
violations, added new images and updated the readme.
Parts:
- added C20: CL05B104JP5NNNC, PCB_Footprints:C0402, symbol CL05B104JP5NNNC
- added R20: RC1005F123CS, PCB_Footprints:R0402, symbol RC1005F123CS
- added R21, R22: RC1005F103CS, PCB_Footprints:R0402, symbol RC1005F103CS
- added SW2: B3U-1000P, PCB_Footprints:B3U-1000P, symbol B3U-1000P
Connections:
- net ESP_PGM_MODE: now also R22.2
- net GND: now also C20.2, R21.2, SW2.1
- net STM_ESP_RST: now also U4.2 (EN), C20.1, R20.2, SW2.2
- net at U4.17 (IO2): now also R21.1
- net +3V3: now reaches C19.1, U4.21 (3V3)
- net +3V3: now also R20.1, R22.1
Other:
- note added: "ESP toggle STM32 Reset"
